File: GSM EMERGENCY/Hardware/maza-gsm.sch (KiCad schematic (older format))
At the start: 1 part

Commit message: Schematics updated
Parts:
- added BT?: Battery_Cell, symbol Battery_Cell
- added C? (x2): 470uF, symbol CP1
- added C?: 100nF, symbol CP1
- added C? (x2): 100nF, symbol C
- added C? (x2): C, symbol C
- added C?: 4.7uF, symbol C
- added C?: 1uF, symbol C
- added C? (x6): 10pF, symbol C
- added C? (x6): 33pF, symbol C
- added D?: 5.1V, symbol D_Zener_Small_ALT
- added D?: D, symbol D
- added D? (x2): ESD, symbol D_Zener_Small_ALT
- added J?: DC_SUPPLY_IN, symbol CONN_01X02
- added MK?: Microphone, symbol Microphone
- added Q?: Q_NPN_BCE, symbol Q_NPN_BCE
- added Q?: BC548, TO_SOT_Packages_THT:TO-92_Molded_Narrow, symbol BC548
- added R?: 51K, symbol R
- added R?: 4.7K, symbol R
- added R? (x2): 47K, symbol R
- added R?: 124K, symbol R
- added R?: 56K, symbol R
- added R?: 470R, symbol R
- added R?: 75K, 1%, symbol R
- added R?: 43K, 1%, symbol R
- added R? (x4): R, symbol R
- added R? (x5): 0R, symbol R
- added R?: 1K, symbol R
- added R?: 5.6K, symbol R
- added U?: MC60, symbol MC60
- added U?: MIC29302_LDO, symbol MIC29302_LDO
- added U?: SGM2019_LDO, symbol SGM2019_LDO
Connections:
- net labels added: BT_ANT, DC_IN, GND, GNSS_VCC, GNSS_VCC_EN, GSM_DEBUG_RXD, GSM_DEBUG_TXD, GSM_ON/OFF, GSM_POWER_BTN, GSM_RXD, GSM_TXD, MICN, MICP, PWRKEY, VBAT, VRTC
- wire segments 0 -> 165
Other:
- note added: "Close to Microphone"
- note added: "Close to Module"
- note added: "DIFFERENTIAL WIRE"
- note added: "Power Supply of the GSM Part"
- note added: "Power supply of GNSS Part in All-in-one Solution"
- note added: "VRTC is Powered by \na Rechargeable Battery\n"

Commit message: Added the pcb file and schematics for GSM section
Parts:
- removed U?: PIC24FJ256GA606, symbol PIC24FJ256GA606
- added C? (x9): 10pF, symbol C
- added C? (x13): 33pF, symbol C
- added C?: 100nF, symbol C
- added C?: 22uF, symbol C
- added C?: 4.7uF, symbol C
- added C? (x4): 10uF, symbol C
- added C?: 0.1uF, symbol C
- added D? (x4): ESD, symbol D_Zener_Small_ALT
- added D? (x3): TVD DIODE, symbol D_ALT
- added D?: TVS DIODE, symbol D_ALT
- added D? (x2): LED, symbol LED_ALT
- added D?: D_Zener_ALT, symbol D_Zener_ALT
- added D?: D_TVS_ALT, symbol D_TVS_ALT
- added J?: PCM CON, symbol CONN_01X04
- added J?: SD CON, symbol CONN_01X03
- added J?: SIM_Card, symbol SIM_Card
- added LS?: 32Ohm,Speaker, symbol Speaker
- added LS?: 8OHM, SPEAKER, symbol Speaker
- added Q?: BC548, TO_SOT_Packages_THT:TO-92_Molded_Narrow, symbol BC548
- added Q?: BC307, TO_SOT_Packages_THT:TO-92_Molded_Narrow, symbol BC307
- added R? (x3): 22R, symbol R
- added R? (x10): 0R, symbol R
- added R? (x2): 4.7K, symbol R
- added R? (x2): 47K, symbol R
- added R? (x2): 300R, symbol R
- added R?: 10K, symbol R
- added U?: Audio_Jack3.3mm, symbol Audio_Jack3.3mm
- added U?: PIC32MX150F128B, symbol PIC32MX150F128B
- J?: value DC_SUPPLY_IN -> DC_SUPPLY_12V_IN
- MK?: value Microphone -> 2.2Kohms, Load Res.Mic
Connections:
- net labels added: 1PPS, 3V3, AGND, LOUDSPKN, LOUDSPKP, NETLIGHT, PCM_CLK, PCM_IN, PCM_OUT, PCM_SYNC, SD_CLK, SD_CMD, SD_DATA, SIM_CLK, SIM_DATA, SIM_GND, SIM_RST, SIM_VDD, SPKN, SPKP, ~MCLR~
- wire segments 165 -> 401
- no-connect marks 0 -> 6
Other:
- note added: "1PPS LED CIRCUIT"
- note added: "AUDIO CIRCUIT"
- note added: "Close to Audio Jack"
- note added: "Close to Speaker"
- note added: "Close to loud Speaker"
- note added: "DIGITAL AUDIO (PCM) INTERFACE"
- note added: "EarPhone Interface"
- note added: "NETWORK LED CIRCUIT"
- note added: "SD CARD INTERFACE"
- note added: "SIM CARD INTERFACE"

Commit message: Added sch for OLED,OSC,PB
Parts:
- removed J?: SIM_Card, symbol SIM_Card
- removed U?: PIC32MX150F128B, symbol PIC32MX150F128B
- added AE? (x3): Antenna, symbol Antenna
- added C? (x6): antenna C, symbol C
- added C? (x4): 33pF, symbol C
- added C? (x3): 100nF, symbol C
- added C? (x8): 100uF, symbol C
- added C?: 47pF, symbol C
- added C? (x2): 33uF,16V, symbol CP
- added C?: 1pF, symbol C
- added C? (x2): 4.7uF, symbol C
- added C?: 10uF, symbol CP
- added C?: 4.7uF, symbol CP
- added C? (x2): C, symbol C
- added D? (x3): TVD DIODE, symbol D_ALT
- added D?: TVS DIODE, symbol D_ALT
- added D?: 1N5817, symbol D_Schottky
- added D?: LED, symbol LED
- added J? (x2): SIM_Card, symbol SIM_Card
- added J?: 12V_IN, symbol CONN_01X02
- added J?: 12V_JMPR, symbol CONN_01X03
- added J?: CONN_01X30, symbol CONN_01X30
- added L?: 18uH, symbol L_Small
- added Q?: BC548, TO_SOT_Packages_THT:TO-92_Molded_Narrow, symbol BC548
- added R? (x5): 0R, symbol R
- added R? (x3): 22R, symbol R
- added R?: 4.7K, symbol R
- added R?: 300R, symbol R
- added R?: 10K, symbol R
- added R?: 3K3, symbol R
- added R?: 820K, symbol R
- added R? (x4): R, symbol R
- added SW? (x4): 2way_push_btn, symbol 2way_push_btn
- added U?: PIC32MX340F256H, symbol PIC32MX340F256H
- added U?: MAX734, symbol MAX734
- added Y?: Crystal, symbol Crystal
Connections:
- net labels added: +3V3, 12V, 12V_EXT, 12V_OUT, GNSS_ANT, OLED_12V_SHDN, OLED_BS1, OLED_BS2, OLED_CS, OLED_D/C, OLED_RST, OLED_SCK, OLED_SDI, OLED_VDD, OLED_VDD_PIN, OSC1, OSC2, PB1, PB2, PB3, PB4, RF_ANT, SIM2_CLK, SIM2_DATA, SIM2_RST, SIM2_VDD
- wire segments 401 -> 649
- no-connect marks 6 -> 30
Other:
- note added: "(optional)"
- note added: "BT ANTENNA CIRCUIT"
- note added: "GNSS ANTENNA CIRCUIT"
- note added: "GNSS SUPPLY Enable"
- note added: "OLED DISPLAY INTERFACE"
- note added: "OSCILLATOR CIRCUIT"
- note added: "PUSH BUTTON INTERFACE"
- note added: "RESET CIRCUIT"
- note added: "RF ANTENNA CIRCUIT"
- note added: "SIM2 CARD INTERFACE"
- note added: "To make GSM module on/off"
- moved on the sheet: C?, D?, J?, Q?, R?, U?

Commit message: sch added TVS doide in SIM interface
Parts:
- removed BT?: Battery_Cell, symbol Battery_Cell
- removed C?: 100uF, symbol C
- removed C? (x2): C, symbol C
- removed C?: 10pF, symbol C
- removed D?: D, symbol D
- removed D? (x6): TVD DIODE, symbol D_ALT
- removed D? (x2): TVS DIODE, symbol D_ALT
- removed J?: DC_SUPPLY_12V_IN, symbol CONN_01X02
- removed J?: SIM_Card, symbol SIM_Card
- removed Q?: Q_NPN_BCE, symbol Q_NPN_BCE
- removed Q? (x3): BC548, TO_SOT_Packages_THT:TO-92_Molded_Narrow, symbol BC548
- removed R? (x2): R, symbol R
- removed R? (x3): 0R, symbol R
- removed U?: PIC32MX340F256H, symbol PIC32MX340F256H
- removed Y?: Crystal, symbol Crystal
- added BT1: Battery_Cell, Connectors_Hirose:Hirose_DF13-02P-1.25DSA_02x1.25mm_Straight, symbol Battery_Cell
- added C10: 10pF, Capacitors_SMD:C_0603_HandSoldering, symbol C
- added C33: 100uF,Tantalum, ESR=0.7Ohm, Capacitors_Tantalum_SMD:CP_Tantalum_Case-X_EIA-7343-43_Hand, symbol CP
- added C69, C76: 4.7uF, Capacitors_SMD:C_0603_HandSoldering, symbol C
- added C74: 15pF, Capacitors_SMD:C_0603_HandSoldering, symbol C
- added C77: 0.1uF, Capacitors_SMD:C_0603_HandSoldering, symbol C
- added C78: 1uF, Capacitors_SMD:C_0603_HandSoldering, symbol C
- added C79: 0.15uF, Capacitors_SMD:C_0603_HandSoldering, symbol C
- added C80, C81: 10uF, Capacitors_SMD:C_0603_HandSoldering, symbol C
- added C82: 0.47uF, Capacitors_SMD:C_0603_HandSoldering, symbol C
- added C83: 33uF, Capacitors_SMD:C_0603_HandSoldering, symbol C
- added C87: CP10uF,Tantalum, ESR=0.7Ohm, Capacitors_Tantalum_SMD:CP_Tantalum_Case-X_EIA-7343-43_Hand, symbol CP
- added D? (x2): TVS_DIODE_CM1224, symbol TVS_DIODE_CM1224
- added J1: SIM_Card, symbol SIM_Card
- added J5: USB_OTG, symbol USB_OTG
- added J6: POWER_ADAPTER, symbol CONN_01X02
- added L1: 1uH, symbol L
- added Q1, Q2, Q4, Q5: PN2222A, TO_SOT_Packages_THT:TO-92_Molded_Narrow, symbol PN2222A
- added R46, R60: 0R, Resistors_SMD:R_0603_HandSoldering, symbol R
- added R48: 10K, Resistors_SMD:R_0603_HandSoldering, symbol R
- added R49, R50, R54, R55: 100K, Resistors_SMD:R_0603_HandSoldering, symbol R
- added R52: 3K, Resistors_SMD:R_0603_HandSoldering, symbol R
- added R53: 1.2K, Resistors_SMD:R_0603_HandSoldering, symbol R
- added TH1: 10K_Thermistor_NTC, symbol Thermistor_NTC
- added U5: MAX8903A, symbol MAX8903A
- added U6: LM3940, symbol LM3940
- added U7: PIC32MX440F512H, symbol PIC32MX440F512H
- added X1: oscillator_DSC1033, symbol oscillator_DSC1033
- C1, C11, C12, C14, C15, C16, C17, C18, C19, C2, C20, C21, C22, C23, C24, C25, C26, C28, C29, C3, C30, C32, C34, C36, C39, C4, C40, C41, C42, C43, C44, C45, C46, C48, C5, C52, C53, C55, C59, C6, C60, C61, C62, C63, C66, C67, C68, C7, C70, C71, C72, C73, C8, C84, C85, C9, C90, C91: renamed from C?; footprint (none) -> Capacitors_SMD:C_0603_HandSoldering
- C13, C31: renamed from C?; value 470uF -> 470uF,E; footprint (none) -> Capacitors_SMD:CP_Elec_3x5.3
- C27: renamed from C?; value 100nF -> 100nF,E; footprint (none) -> Capacitors_SMD:CP_Elec_3x5.3
- C35: renamed from C?; value 100uF -> 100nF; footprint (none) -> Capacitors_SMD:C_0603_HandSoldering
- C37: renamed from C?; value 100uF -> 10pF; footprint (none) -> Capacitors_SMD:C_0603_HandSoldering
- C38: renamed from C?; value 100uF -> 33pF; footprint (none) -> Capacitors_SMD:C_0603_HandSoldering
- C47, C54: renamed from C?; value 10uF -> 33pF; footprint (none) -> Capacitors_SMD:C_0603_HandSoldering
- C64: renamed from C?; value C -> 10uF; footprint (none) -> Capacitors_SMD:C_0603_HandSoldering
- C65: renamed from C?; value C -> 100nF; footprint (none) -> Capacitors_SMD:C_0603_HandSoldering
- C86: renamed from C?; footprint (none) -> Capacitors_SMD:CP_Elec_3x5.3
- C88: renamed from C?; value 33uF,16V -> 33uF,16V,E; footprint (none) -> Capacitors_SMD:CP_Elec_3x5.3
- C89: renamed from C?; value 4.7uF -> 4.7uF,16V,E; footprint (none) -> Capacitors_SMD:CP_Elec_3x5.3
- C92: renamed from C?; value 10uF -> 10uF,16V,E; footprint (none) -> Capacitors_SMD:CP_Elec_3x5.3
- D12: renamed from D?; value 5.1V -> 5.1V Zener
- D13, D21: renamed from D?; footprint (none) -> LEDs:LED_0805
- R1, R10, R11, R12, R13, R14, R15, R16, R17, R18, R19, R2, R20, R21, R22, R23, R24, R25, R26, R27, R28, R29, R3, R30, R31, R35, R36, R37, R38, R39, R4, R40, R45, R5, R56, R57, R58, R59, R6, R61, R7, R8, R9: renamed from R?; footprint (none) -> Resistors_SMD:R_0603_HandSoldering
- R32, R33, R34: renamed from R?; value 0R -> 1K; footprint (none) -> Resistors_SMD:R_0603_HandSoldering
- R41: renamed from R?; value R -> 4.7K; footprint (none) -> Resistors_SMD:R_0603_HandSoldering
- R42: renamed from R?; value R -> 47K; footprint (none) -> Resistors_SMD:R_0603_HandSoldering
- R43, R44, R47, R51: renamed from R?; value R -> 10K; footprint (none) -> Resistors_SMD:R_0603_HandSoldering
- gave numbers to parts that had none: 39
Connections:
- net labels added: BAT, BT_CHRG_IND, BT_DOK, BT_FLT, BT_UOK, CBST_LX, OSC, SIM1_CH1, SIM1_CH2, SIM1_CH3, SIM1_CH4, SIM1_VDD, SIM2_CH1, SIM2_CH2, SIM2_CH3, SIM2_CH4, THM, USB_ADAPTER, USB_D+, USB_D-, USB_ID, VBUS, VCORE, VL, VSYS
- net labels removed: +3V3, AGND, DC_IN, OSC1, OSC2, SIM_VDD, VRTC
- wire segments 649 -> 798
- no-connect marks 30 -> 53
Other:
- note added: "3.3 V REGULATOR"
- note added: "CHARGEING CIRCUIT"
- note added: "DIGITAL AUDIO \n(PCM) INTERFACE"
- note added: "POWER SWITCH FOR GSM MODULE"
- note added: "Place near VCORE and VSS\n"
- note removed: "DIGITAL AUDIO (PCM) INTERFACE"
- note removed: "VRTC is Powered by \na Rechargeable Battery\n"
- moved on the sheet: C35, C37, C38, C48, C61, C63, C64, C65, C68, C70, C71, C72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

Commit message: Completed till schematics
Parts:
- removed AE2, AE3: Antenna, symbol Antenna
- removed D12: 5.1V Zener, symbol D_Zener_Small_ALT
- removed R48: 10K, Resistors_SMD:R_0603_HandSoldering, symbol R
- removed TH1: 10K_Thermistor_NTC, symbol Thermistor_NTC
- added D14, D15, D16, D17, D18, D21, D22, D23: LED, LEDs:LED_1206, symbol LED_ALT
- added D9: 5.1V Zener, Diodes_SMD:D_SOD-123, symbol D_Zener
- added F1, F2: IPEX_CON, kicad_libraries:IPEX_CON_MHF, symbol IPEX_CON-RESCUE-maza-gsm
- added Q11, Q12, Q13, Q5, Q6, Q7, Q8, Q9: PN2222A, TO_SOT_Packages_THT:TO-92_Molded_Narrow, symbol PN2222A
- added R54, R58, R61, R65, R69, R73, R77, R82: 4.7K, Resistors_SMD:R_0805_HandSoldering, symbol R
- added R56, R59, R62, R66, R70, R74, R78, R83: 47K, Resistors_SMD:R_0805_HandSoldering, symbol R
- added R57, R60, R63, R67, R72, R76, R80, R84: 300R, Resistors_SMD:R_0805_HandSoldering, symbol R
- AE1: footprint (none) -> kicad_libraries:GSM_ANTENNA_Yageo_ANT2112A010B0918A
- C1, C10, C11, C12, C14, C15, C16, C17, C18, C19, C2, C20, C21, C22, C23, C24, C25, C26, C28, C29, C3, C30, C32, C34, C35, C36, C37, C38, C39, C4, C40, C41, C42, C43, C44, C45, C46, C47, C48, C5, C52, C53, C54, C55, C59, C6, C60, C61, C62, C63, C64, C65, C66, C67, C68, C69, C7, C70, C71, C72, C73, C74, C8, C9: footprint Capacitors_SMD:C_0603_HandSoldering -> Capacitors_SMD:C_0805_HandSoldering
- C49, C50, C51, C56, C57, C58: footprint (none) -> Capacitors_SMD:C_0805_HandSoldering
- C75: renamed from C76; footprint Capacitors_SMD:C_0603_HandSoldering -> Capacitors_SMD:C_0805_HandSoldering
- C76: renamed from C77; footprint Capacitors_SMD:C_0603_HandSoldering -> Capacitors_SMD:C_0805_HandSoldering
- C77: renamed from C78; footprint Capacitors_SMD:C_0603_HandSoldering -> Capacitors_SMD:C_0805_HandSoldering
- C78: renamed from C79; footprint Capacitors_SMD:C_0603_HandSoldering -> Capacitors_SMD:C_0805_HandSoldering
- C79: renamed from C80; footprint Capacitors_SMD:C_0603_HandSoldering -> Capacitors_SMD:C_0805_HandSoldering
- C80: renamed from C81; footprint Capacitors_SMD:C_0603_HandSoldering -> Capacitors_SMD:C_0805_HandSoldering
- C81: renamed from C82; footprint Capacitors_SMD:C_0603_HandSoldering -> Capacitors_SMD:C_0805_HandSoldering
- C82: renamed from C83; footprint Capacitors_SMD:C_0603_HandSoldering -> Capacitors_SMD:C_0805_HandSoldering
- C83: renamed from C84; footprint Capacitors_SMD:C_0603_HandSoldering -> Capacitors_SMD:C_0805_HandSoldering
- C84: renamed from C85; footprint Capacitors_SMD:C_0603_HandSoldering -> Capacitors_SMD:C_0805_HandSoldering
- C89: renamed from C90; footprint Capacitors_SMD:C_0603_HandSoldering -> Capacitors_SMD:C_0805_HandSoldering
- C90: renamed from C91; footprint Capacitors_SMD:C_0603_HandSoldering -> Capacitors_SMD:C_0805_HandSoldering
- D1, D12: renamed from D?; footprint (none) -> kicad_libraries:CM1224-4SO-SOT23
- D10: renamed from D13; footprint LEDs:LED_0805 -> LEDs:LED_0603
- D11: renamed from D14; footprint (none) -> Diodes_SMD:D_SOD-123
- D13: renamed from D15; footprint (none) -> Diodes_SMD:D_SOD-123
- D19: renamed from D20; value 1N5817 -> SS14FL; footprint (none) -> kicad_libraries:SChottky-diode-SS14FL-Fairchild
- D2, D3, D4, D5, D6, D7: footprint (none) -> Diodes_SMD:D_SOD-123
- D20: renamed from D21; footprint LEDs:LED_0805 -> LEDs:LED_0603
- D8: footprint (none) -> LEDs:LED_1206
- J1, J4: footprint (none) -> kicad_libraries:MICRO-SIM-78646-3001-MOLEX
- J2: footprint (none) -> Pin_Headers:Pin_Header_Angled_1x04_Pitch2.54mm
- J3: footprint (none) -> Pin_Headers:Pin_Header_Angled_1x03_Pitch2.54mm
- J5: footprint (none) -> Connectors:USB_Micro-B_10103594-0001LF
- J6: footprint (none) -> Connectors:bornier2
- J7: footprint (none) -> Socket_Strips:Socket_Strip_Straight_1x02_Pitch2.54mm
- J8: footprint (none) -> Socket_Strips:Socket_Strip_Straight_1x03_Pitch2.54mm
- J9: footprint (none) -> Connectors_Molex:Molex_Panelmate-53780-3070_30x1.25mm_Angled
- L1, L2: footprint (none) -> Inductors_SMD:L_0805_HandSoldering
- LS1, LS2, MK1: footprint (none) -> Capacitors_SMD:C_1206_HandSoldering
- R1, R10, R11, R12, R13, R14, R15, R16, R17, R18, R19, R2, R20, R21, R22, R23, R24, R25, R26, R27, R28, R29, R3, R30, R31, R32, R33, R34, R35, R36, R37, R38, R39, R4, R40, R41, R42, R43, R44, R45, R46, R47, R5, R55, R6, R7, R8, R9: footprint Resistors_SMD:R_0603_HandSoldering -> Resistors_SMD:R_0805_HandSoldering
- R48: renamed from R49; footprint Resistors_SMD:R_0603_HandSoldering -> Resistors_SMD:R_0805_HandSoldering
- R49: renamed from R50; footprint Resistors_SMD:R_0603_HandSoldering -> Resistors_SMD:R_0805_HandSoldering
- R50: renamed from R51; footprint Resistors_SMD:R_0603_HandSoldering -> Resistors_SMD:R_0805_HandSoldering
- R51: renamed from R52; footprint Resistors_SMD:R_0603_HandSoldering -> Resistors_SMD:R_0805_HandSoldering
- R52: renamed from R53; footprint Resistors_SMD:R_0603_HandSoldering -> Resistors_SMD:R_0805_HandSoldering
- R53: renamed from R54; footprint Resistors_SMD:R_0603_HandSoldering -> Resistors_SMD:R_0805_HandSoldering
- R64: renamed from R56; footprint Resistors_SMD:R_0603_HandSoldering -> Resistors_SMD:R_0805_HandSoldering
- R68: renamed from R57; footprint Resistors_SMD:R_0603_HandSoldering -> Resistors_SMD:R_0805_HandSoldering
- R71: renamed from R58; footprint Resistors_SMD:R_0603_HandSoldering -> Resistors_SMD:R_0805_HandSoldering
- R75: renamed from R59; footprint Resistors_SMD:R_0603_HandSoldering -> Resistors_SMD:R_0805_HandSoldering
- R79: renamed from R60; footprint Resistors_SMD:R_0603_HandSoldering -> Resistors_SMD:R_0805_HandSoldering
- R81: renamed from R61; footprint Resistors_SMD:R_0603_HandSoldering -> Resistors_SMD:R_0805_HandSoldering
- SW1, SW2, SW3, SW4: footprint (none) -> kicad_libraries:Push_Btn_DPDT_ESB3313_Panasonic
- U1: footprint (none) -> TO_SOT_Packages_SMD:TO-263-5Lead
- U2: footprint (none) -> kicad_libraries:MC60-Quectel
- U3: footprint (none) -> TO_SOT_Packages_SMD:SOT-23-5_HandSoldering
- U4: footprint (none) -> kicad_libraries:Audio_Jack_3.5mm
- U5: footprint (none) -> Housings_DFN_QFN:QFN-28-1EP_4x4mm_Pitch0.4mm
- U6: footprint (none) -> TO_SOT_Packages_SMD:SOT-223
- U7: footprint (none) -> kicad_libraries:TQFP_64-10mmX10mm
- U8: footprint (none) -> kicad_libraries:SO-8
- X1: footprint (none) -> kicad_libraries:OSC_DS1033
- renumbered C86 to C85, C87 to C86, C88 to C87, C89 to C88, C92 to C91, Q5 to Q10
Connections:
- net labels added: LED1, LED2, LED3, LED4, LED5, LED6, LED7, LED8
- net labels removed: THM
- wire segments 798 -> 890
- no-connect marks 53 -> 45
Other:
- note added: "GPP LED CIRCUIT"

Commit message: Added the Accelerometer in sch.
Parts:
- removed C27: 100nF,E, Capacitors_SMD:CP_Elec_3x5.3, symbol CP1
- removed D10: LED, LEDs:LED_0603, symbol LED_ALT
- removed D13: D_Zener_ALT, Diodes_SMD:D_SOD-123, symbol D_Zener_ALT
- removed D14, D15, D16, D17, D18, D21, D22, D23, D8: LED, LEDs:LED_1206, symbol LED_ALT
- removed D20: LED, LEDs:LED_0603, symbol LED
- removed J7: 12V_IN, Socket_Strips:Socket_Strip_Straight_1x02_Pitch2.54mm, symbol CONN_01X02
- removed J8: 12V_JMPR, Socket_Strips:Socket_Strip_Straight_1x03_Pitch2.54mm, symbol CONN_01X03
- removed LS1: 32Ohm,Speaker, Capacitors_SMD:C_1206_HandSoldering, symbol Speaker
- removed LS2: 8OHM, SPEAKER, Capacitors_SMD:C_1206_HandSoldering, symbol Speaker
- removed MK1: 2.2Kohms, Load Res.Mic, Capacitors_SMD:C_1206_HandSoldering, symbol Microphone
- removed Q1, Q10, Q11, Q12, Q13, Q2, Q4, Q5, Q6, Q7, Q8, Q9: PN2222A, TO_SOT_Packages_THT:TO-92_Molded_Narrow, symbol PN2222A
- removed Q3: BC307, TO_SOT_Packages_THT:TO-92_Molded_Narrow, symbol BC307
- removed R56, R59, R74: 47K, Resistors_SMD:R_0805_HandSoldering, symbol R
- removed R58, R61, R69: 4.7K, Resistors_SMD:R_0805_HandSoldering, symbol R
- removed R76, R80, R84: 300R, Resistors_SMD:R_0805_HandSoldering, symbol R
- removed SW1, SW2, SW3, SW4: 2way_push_btn, kicad_libraries:Push_Btn_DPDT_ESB3313_Panasonic, symbol 2way_push_btn
- removed U4: Audio_Jack3.3mm, kicad_libraries:Audio_Jack_3.5mm, symbol Audio_Jack3.3mm
- added C27: 100nF, Capacitors_SMD:C_0805_HandSoldering, symbol C
- added C? (x4): 0.1uF, symbol C
- added C?: 4.7uF, symbol C
- added D11: D_TVS_ALT, Diodes_SMD:D_SOD-123, symbol D_TVS_ALT
- added J10: ON_OFF_SWITCH, Connectors_Terminal_Blocks:TerminalBlock_Pheonix_MPT-2.54mm_3pol, symbol CONN_01X03
- added J11: LED2, Connectors_Terminal_Blocks:TerminalBlock_Pheonix_MPT-2.54mm_2pol, symbol CONN_01X02
- added J12: LED3, Connectors_Terminal_Blocks:TerminalBlock_Pheonix_MPT-2.54mm_2pol, symbol CONN_01X02
- added J13: LED4, Connectors_Terminal_Blocks:TerminalBlock_Pheonix_MPT-2.54mm_2pol, symbol CONN_01X02
- added J14: LED5, Connectors_Terminal_Blocks:TerminalBlock_Pheonix_MPT-2.54mm_2pol, symbol CONN_01X02
- added J15: LED6, Connectors_Terminal_Blocks:TerminalBlock_Pheonix_MPT-2.54mm_2pol, symbol CONN_01X02
- added J16: LED7, Connectors_Terminal_Blocks:TerminalBlock_Pheonix_MPT-2.54mm_2pol, symbol CONN_01X02
- added J17: LED8, Connectors_Terminal_Blocks:TerminalBlock_Pheonix_MPT-2.54mm_2pol, symbol CONN_01X02
- added J19: PB1, Pin_Headers:Pin_Header_Straight_1x02_Pitch2.54mm, symbol CONN_01X02
- added J2: NETWORK_LED, Connectors_Terminal_Blocks:TerminalBlock_Pheonix_MPT-2.54mm_2pol, symbol CONN_01X02
- added J20: PB2, Pin_Headers:Pin_Header_Straight_1x02_Pitch2.54mm, symbol CONN_01X02
- added J21: PB3, Pin_Headers:Pin_Header_Straight_1x02_Pitch2.54mm, symbol CONN_01X02
- added J22: PB4, Pin_Headers:Pin_Header_Straight_1x02_Pitch2.54mm, symbol CONN_01X02
- added J23: OLED_INDICATOR, Pin_Headers:Pin_Header_Straight_1x02_Pitch2.54mm, symbol CONN_01X02
- added J24: 32Ohm,Speaker, Pin_Headers:Pin_Header_Straight_1x02_Pitch2.54mm, symbol CONN_01X02
- added J25: 8OHM, SPEAKER, Pin_Headers:Pin_Header_Straight_1x02_Pitch2.54mm, symbol CONN_01X02
- added J26: 2.2Kohms, Load Res.Mic, Pin_Headers:Pin_Header_Straight_1x02_Pitch2.54mm, symbol CONN_01X02
- added J27: ICSP, Pin_Headers:Pin_Header_Straight_1x05_Pitch2.54mm, symbol CONN_01X05
- added J5: 1PPS_LED, Connectors_Terminal_Blocks:TerminalBlock_Pheonix_MPT-2.54mm_2pol, symbol CONN_01X02
- added J9: LED1, Connectors_Terminal_Blocks:TerminalBlock_Pheonix_MPT-2.54mm_2pol, symbol CONN_01X02
- added Q1, Q10, Q11, Q12, Q13, Q2, Q4, Q5, Q6, Q7, Q8, Q9: BC847, TO_SOT_Packages_SMD:SOT-23_Handsoldering, symbol BC847
- added Q3: BC857, TO_SOT_Packages_SMD:SOT-23_Handsoldering, symbol BC857
- added R44, R48, R50, R55, R88: 0R, Resistors_SMD:R_0805_HandSoldering, symbol R
- added R64, R71, R75, R79, R89: 300R, Resistors_SMD:R_0805_HandSoldering, symbol R
- added R68, R81, R85: 4.7K, Resistors_SMD:R_0805_HandSoldering, symbol R
- added R87: 47K, Resistors_SMD:R_0805_HandSoldering, symbol R
- added R? (x4): R, symbol R
- added U4: Audio_Jack3.5mm, kicad_libraries:Audio_Jack_3.5mm, symbol Audio_Jack3.5mm
- added U?: ACCELEROMETER_FXOS8700CQ_NXP, symbol ACCELEROMETER_FXOS8700CQ_NXP
- BT1: footprint Connectors_Hirose:Hirose_DF13-02P-1.25DSA_02x1.25mm_Straight -> Pin_Headers:Pin_Header_Straight_1x02_Pitch2.54mm
- C13, C31: footprint Capacitors_SMD:CP_Elec_3x5.3 -> Capacitors_SMD:CP_Elec_10x10.5
- C49, C50, C51, C56, C57, C58: value antenna C -> NM C
- C86: footprint Capacitors_Tantalum_SMD:CP_Tantalum_Case-X_EIA-7343-43_Hand -> Capacitors_Tantalum_SMD:CP_Tantalum_Case-A_EIA-3216-18_Hand
- C88: footprint Capacitors_SMD:CP_Elec_3x5.3 -> Capacitors_SMD:CP_Elec_4x5.3
- C91: footprint Capacitors_SMD:CP_Elec_3x5.3 -> Capacitors_SMD:CP_Elec_5x5.3
- J18: renamed from J9; value CONN_01X30 -> OLED CONNECTOR
- J3: renamed from J2; footprint Pin_Headers:Pin_Header_Angled_1x04_Pitch2.54mm -> Pin_Headers:Pin_Header_Straight_1x04_Pitch2.54mm
- J4: renamed from J3; footprint Pin_Headers:Pin_Header_Angled_1x03_Pitch2.54mm -> Pin_Headers:Pin_Header_Straight_1x03_Pitch2.54mm
- J8: renamed from J6; footprint Connectors:bornier2 -> Connectors_Terminal_Blocks:TerminalBlock_Pheonix_MPT-2.54mm_2pol
- R60, R63: value 300R -> 47K
- R62: value 47K -> 4.7K
- R72: value 300R -> 4.7K
- R73, R82: value 4.7K -> 47K
- R83: value 47K -> 300R
- renumbered D12 to D10, D19 to D12, D9 to D8, D11 to D9, J4 to J6, J5 to J7, R44 to R45, R45 to R46, R46 to R47, R47 to R49, R48 to R51, R49 to R52, R50 to R53, R51 to R54, R52 to R56, R53 to R57, R54 to R58, R55 to R59, R57 to R61, R64 to R69, R68 to R74, R71 to R76, R75 to R80, R79 to R84, R81 to R86
Connections:
- net labels added: INT1, INT2, PGEC2, PGED2, SA0/MISO, SCL/SCLK, SDA/MOSI, VDDIO, ~ACC_CS~
- net labels removed: 12V_EXT, 12V_OUT
- wire segments 890 -> 932
- no-connect marks 45 -> 44
Other:
- note added: "ICSP connector\n"
- moved on the sheet: R76, R9, U2, U7
