File: GSM EMERGENCY/Hardware/V1/maza-gsm.sch (KiCad schematic (older format))
At the start: 259 parts, among them J1 SIM_Card, J10 ON_OFF_SWITCH, J11 LED2, J12 LED3, J13 LED4, J14 LED5, J15 LED6, J16 LED7, J17 LED8, J18 OLED CONNECTOR, J19 PB1, J2 NETWORK_LED, J20 PB2, J21 PB3, J22 PB4, J23 OLED_INDICATOR, J24 32Ohm,Speaker, J25 8OHM, SPEAKER, J26 2.2Kohms, Load Res.Mic, J27 ICSP, J3 PCM CON, J4 SD CON, J5 1PPS_LED, J6 SIM_Card, J7 USB_OTG, J8 POWER_ADAPTER, J9 LED1, P1 TH_PAD, P2 TH_PAD, P3 TH_PAD, P4 TH_PAD, P5 TH_PAD, P6 TH_PAD, P7 TH_PAD, P8 TH_PAD, Q1 BC847, Q10 BC847, Q11 BC847, Q12 BC847, Q13 BC847, Q2 BC847, Q3 BC857, Q4 BC847, Q5 BC847, Q6 BC847, Q7 BC847, Q8 BC847, Q9 BC847, U1 MIC29302_LDO, U2 MC60, U3 SGM2019_LDO, U4 Audio_Jack3.5mm, U5 MAX8903A, U6 LM3940, U7 PIC32MX440F512H, U8 MAX734, U9 ADXL_335, X1 oscillator_DSC1033

Commit message: PCB completed
Parts:
- removed C10, C11, C12: 10pF, Capacitors_SMD:C_0805_HandSoldering, symbol C
- removed C24, C25, C26, C55, C59, C60, C62: 33pF, Capacitors_SMD:C_0805_HandSoldering, symbol C
- removed C66, C67: 100nF, Capacitors_SMD:C_0805_HandSoldering, symbol C
- removed D10: TVS_DIODE_CM1224, kicad_libraries:CM1224-4SO-SOT23, symbol TVS_DIODE_CM1224
- removed D6, D7: ESD, Diodes_SMD:D_SOD-123, symbol D_Zener_Small_ALT
- removed J12: LED3, Resistors_SMD:R_0805_HandSoldering, symbol CONN_01X02
- removed J15: LED6, Resistors_SMD:R_0805_HandSoldering, symbol CONN_01X02
- removed J25: 8OHM, SPEAKER, Pin_Headers:Pin_Header_Straight_1x02_Pitch2.54mm, symbol CONN_01X02
- removed J3: PCM CON, Pin_Headers:Pin_Header_Straight_1x04_Pitch2.54mm, symbol CONN_01X04
- removed J4: SD CON, Pin_Headers:Pin_Header_Straight_1x03_Pitch2.54mm, symbol CONN_01X03
- removed J6: SIM_Card, kicad_libraries:MICRO-SIM-78646-3001-MOLEX, symbol SIM_Card
- removed P7, P8: TH_PAD, kicad_libraries:TH_HOLE_PAD_6.5mm, symbol TH_PAD
- removed Q11, Q7: BC847, TO_SOT_Packages_SMD:SOT-23_Handsoldering, symbol BC847
- removed R1, R2, R6, R7: 0R, Resistors_SMD:R_0805_HandSoldering, symbol R
- removed R38, R39, R40: 22R, Resistors_SMD:R_0805_HandSoldering, symbol R
- removed R65, R77: 4.7K, Resistors_SMD:R_0805_HandSoldering, symbol R
- removed R66, R78: 47K, Resistors_SMD:R_0805_HandSoldering, symbol R
- removed R67, R79: 300R, Resistors_SMD:R_0805_HandSoldering, symbol R
- J13: value LED4 -> LED3
- J14: value LED5 -> LED4
- J16: value LED7 -> LED5
- J17: value LED8 -> LED6
- J2, J5: footprint Connectors_Terminal_Blocks:TerminalBlock_Pheonix_MPT-2.54mm_2pol -> Resistors_SMD:R_0805_HandSoldering
- J23: footprint Pin_Headers:Pin_Header_Straight_1x02_Pitch2.54mm -> LEDs:LED_0805
- J24, J26: footprint Pin_Headers:Pin_Header_Straight_1x02_Pitch2.54mm -> Resistors_SMD:R_0805_HandSoldering
Connections:
- net labels added: MIC_N, MIC_P, SPK_N, SPK_P, USB_D_+, USB_D_-
- net labels removed: LED7, LED8, LOUDSPKN, MICN, MICP, PCM_CLK, PCM_IN, PCM_OUT, PCM_SYNC, SD_CLK, SD_CMD, SD_DATA, SIM2_CH1, SIM2_CH2, SIM2_CH3, SIM2_CH4, SPKN, SPKP, USB_D+, USB_D-
- wire segments 914 -> 790
- no-connect marks 53 -> 59
Other:
- note removed: "(optional)"
- note removed: "DIGITAL AUDIO \n(PCM) INTERFACE"
- note removed: "SD CARD INTERFACE"
- note removed: "SIM2 CARD INTERFACE"
