File: GSM EMERGENCY/Hardware/V1/maza-gsm.kicad_pcb (KiCad board)
At the start: 2 copper layers, 61 x 113 mm, 221 parts, among them J1 SIM_Card, J10 ON_OFF_SWITCH, J11 LED2, J13 LED3, J14 LED4, J16 LED5, J17 LED6, J18 OLED CONNECTOR, J19 PB1, J2 NETWORK_LED, J20 PB2, J21 PB3, J22 PB4, J23 OLED_INDICATOR, J24 32Ohm,Speaker, J26 2.2Kohms, Load Res.Mic, J27 ICSP, J5 1PPS_LED, J7 USB_OTG, J8 POWER_ADAPTER, J9 LED1, P1 TH_PAD, P2 TH_PAD, P3 TH_PAD, P4 TH_PAD, P5 TH_PAD, P6 TH_PAD, Q1 BC847, Q10 BC847, Q12 BC847, Q13 BC847, Q2 BC847, Q3 BC857, Q4 BC847, Q5 BC847, Q6 BC847, Q8 BC847, Q9 BC847, U1 MIC29302_LDO, U2 MC60, U3 SGM2019_LDO, U4 Audio_Jack3.5mm, U5 MAX8903A, U6 LM3940, U7 PIC32MX440F512H, U8 MAX734, U9 ADXL_335, X1 oscillator_DSC1033

Commit message: Firmware baseline v1
Other:
- board text removed: "1PPS LED CIRCUIT"
- board text removed: "3.3 V REGULATOR"
- board text removed: "AUDIO CIRCUIT"
- board text removed: "BT ANTENNA CIRCUIT GNSS ANTENNA CIRCUIT"
- board text removed: "EarPhone Interface"
- board text removed: "GPP LED CIRCUIT"
- board text removed: "NETWORK LED CIRCUIT"
- board text removed: "OLED DISPLAY INTERFACE"
- board text removed: "POWER SWITCH FOR GSM MODULE"
- board text removed: "Power Supply of the GSM Part"
- board text removed: "Power supply of GNSS Part in All-in-one Solution"
- board text removed: "RESET CKT"
- board text removed: "RF ANTENNA CIRCUIT"
- board text removed: "SIM CARD INTERFACE"
Changed lines of the file:
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@@
     (links 460)
     (no_connects 0)
-    (area 191.924999 35.924999 253.075001 149.075001)
+    (area -62.878572 -62.603572 272.260714 197.625)
     (thickness 1.6)
-    (drawings 22)
+    (drawings 8)
     (tracks 3293)
     (zones 0)
@@
   (page A4)
   (layers
-    (0 F.Cu signal hide)
-    (31 B.Cu signal hide)
+    (0 F.Cu signal)
+    (31 B.Cu signal)
     (32 B.Adhes user)
-    (33 F.Adhes user hide)
+    (33 F.Adhes user)
     (34 B.Paste user)
     (35 F.Paste user hide)
     (36 B.SilkS user)
-    (37 F.SilkS user hide)
+    (37 F.SilkS user)
     (38 B.Mask user)
     (39 F.Mask user hide)
-    (40 Dwgs.User user hide)
+    (40 Dwgs.User user)
     (41 Cmts.User user)
     (42 Eco1.User user)
@@
     (45 Margin user hide)
     (46 B.CrtYd user)
-    (47 F.CrtYd user hide)
+    (47 F.CrtYd user)
     (48 B.Fab user)
-    (49 F.Fab user hide)
+    (49 F.Fab user)
   )
   (setup
@@
     (aux_axis_origin 223 81)
     (grid_origin 223 81)
-    (visible_elements FFFEBFDF)
+    (visible_elements FFFEFFDF)
     (pcbplotparams
       (layerselection 0x00030_80000001)
@@
   (gr_line (start 192 42) (end 192 142) (angle 90) (layer Edge.Cuts) (width 0.15))
   (gr_line (start 198 36) (end 192 42) (angle 90) (layer Edge.Cuts) (width 0.15))
-  (gr_text "RESET CKT" (at 266.225 97.875) (layer F.Fab)
-    (effects (font (size 1.5 1.5) (thickness 0.3)))
-  )
-  (gr_text "OLED DISPLAY \nINTERFACE" (at 177.675 -54.175 90) (layer F.Fab)
-    (effects (font (size 1.5 1.5) (thickness 0.3)))
-  )
-  (gr_text "GPP LED CIRCUIT" (at -35.1 27.75) (layer F.Fab)
-    (effects (font (size 1.5 1.5) (thickness 0.3)))
-  )
-  (gr_text "AUDIO CIRCUIT" (at 1.2 133.1) (layer F.Fab)
-    (effects (font (size 1.5 1.5) (thickness 0.3)))
-  )
-  (gr_text "EarPhone Interface" (at 58.6 148) (layer F.Fab)
-    (effects (font (size 1.5 1.5) (thickness 0.3)))
-  )
-  (gr_text "RF ANTENNA CIRCUIT" (at 26.2 105.3) (layer F.Fab)
-    (effects (font (size 1.5 1.5) (thickness 0.3)))
-  )
-  (gr_text "1PPS LED\n CIRCUIT" (at -25.85 5.2) (layer F.Fab)
-    (effects (font (size 1.5 1.5) (thickness 0.3)))
-  )
-  (gr_text "POWER SWITCH \nFOR GSM MODULE" (at 162.02 141.16) (layer F.Fab)
-    (effects (font (size 1.5 1.5) (thickness 0.3)))
-  )
-  (gr_text "BT ANTENNA CIRCUIT\nGNSS ANTENNA CIRCUIT" (at 72.25 102.95) (layer F.Fab)
-    (effects (font (size 1.5 1.5) (thickness 0.3)))
-  )
-  (gr_text "NETWORK LED CIRCUIT" (at -50.2 1.7) (layer F.Fab)
-    (effects (font (size 1.5 1.5) (thickness 0.3)))
-  )
-  (gr_text "SIM CARD INTERFACE" (at 196.55 129.8) (layer F.Fab)
-    (effects (font (size 1.5 1.5) (thickness 0.3)))
-  )
-  (gr_text "3.3 V REGULATOR" (at 163.04 127.51) (layer F.Fab)
-    (effects (font (size 1.5 1.5) (thickness 0.3)))
-  )
-  (gr_text "Power Supply of \nthe GSM Part" (at 70 195) (layer F.Fab)
-    (effects (font (size 1.5 1.5) (thickness 0.3)))
-  )
-  (gr_text "Power supply of GNSS Part\n in All-in-one Solution" (at 158.375 192.05) (layer F.Fab)
-    (effects (font (size 1.5 1.5) (thickness 0.3)))
-  )
   (segment (start 202.795 95.66) (end 201.88 94.745) (width 0.25) (layer F.Cu) (net 1))
   (segment (start 201.88 94.745) (end 201.005 94.745) (width 0.25) (layer F.Cu) (net 1))
